Commit message: add self made maze world

File: sjtu_drone_description/urdf/sjtu_drone.urdf.xacro (robot description, xacro)
@@ -4,4 +4,7 @@
   <!-- Need argument to get from launch file -->
   <xacro:arg name="params_path" default="$(find sjtu_drone_bringup)/config/drone.yaml"/>
+  <xacro:arg name="x" default="0"/>
+  <xacro:arg name="y" default="0"/>
+  <xacro:arg name="z" default="0.04"/>
   <!-- Need seperate property for xacro inorder processing -->
   <xacro:property name="params_path" value="$(arg params_path)"/>
@@ -22,5 +25,5 @@
     </inertial>
     <collision name="sjtu_drone_collision">
-      <origin rpy="0 0 0" xyz="0   0   0.04"/>
+      <origin rpy="0 0 0" xyz="$(arg x) $(arg y) $(arg z)"/>
       <geometry>
         <mesh filename="file://$(find sjtu_drone_description)/models/sjtu_drone/quadrotor_4.stl"/>
@@ -29,5 +32,5 @@
     </collision>
     <visual name="sjtu_drone_visual">
-      <origin rpy="0 0 0" xyz="0   0   0.04"/>
+      <origin rpy="0 0 0" xyz="$(arg x) $(arg y) $(arg z)" />
       <geometry>
         <mesh filename="file://$(find sjtu_drone_description)/models/sjtu_drone/quadrotor_4.dae"/>
@@ -43,5 +46,5 @@
   <link name="sonar_link"/>
   <joint name="front_cam_joint" type="fixed">
-    <origin rpy="0 0 0" xyz="0.2 0 0"/>
+    <origin rpy="0 0 0" xyz="0.2 0 0.45"/>
     <parent link="base_link" />
     <child link="front_cam_link" />
@@ -194,6 +197,6 @@
         <camera_name>front</camera_name>
         <hack_baseline>0.07</hack_baseline>
-        <min_depth>0.2</min_depth>
-        <max_depth>8.0</max_depth>
+        <!-- <min_depth>0.2</min_depth>
+        <max_depth>8.0</max_depth> -->
       </plugin>
     </sensor>
