Commit message: add maze world

File: sjtu_drone_description/urdf/sjtu_drone.urdf (robot description, URDF)
Before this commit: robot sjtu_drone, 5 links, 4 joints
Links:
- link base_link: geometry collision mesh filename=file:///home/carlios/dev_ws/install/sjtu_drone_description/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; visual mesh filename=file:///home/carlios/dev_ws/install/sjtu_drone_description/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

Commit message: add front depth camera

File: sjtu_drone_description/urdf/sjtu_drone.urdf (robot description, URDF)
Before this commit: robot sjtu_drone, 5 links, 4 joints
Links:
- removed link bottom_cam_link
Joints:
- removed joint bottom_cam_joint

File: sjtu_drone_description/urdf/sjtu_drone.urdf.xacro (robot description, xacro)
@@ -48,10 +48,10 @@
   </joint>
   <link name="front_cam_link"/>
-  <joint name="bottom_cam_joint" type="fixed">
+  <!-- <joint name="bottom_cam_joint" type="fixed">
     <origin rpy="0 ${M_PI/2} 0" xyz="0 0 0"/>
     <parent link="base_link" />
     <child link="bottom_cam_link" />
   </joint>
-  <link name="bottom_cam_link"/>
+  <link name="bottom_cam_link"/> -->
   <gazebo>
     <plugin name='simple_drone' filename='libplugin_drone.so'>
@@ -62,7 +62,7 @@
         <remapping>sonar:=sonar</remapping>
         <remapping>camera_front:=camera_front</remapping>
-        <remapping>camera_bottom:=camera_bottom</remapping>
+        <!-- <remapping>camera_bottom:=camera_bottom</remapping> -->
         <remapping>camera_front_info:=camera_front_info</remapping>
-        <remapping>camera_bottom_info:=camera_bottom_info</remapping>
+        <!-- <remapping>camera_bottom_info:=camera_bottom_info</remapping> -->
         <remapping>gps:=gps</remapping>
       </ros>
@@ -171,4 +171,33 @@
   </gazebo>
   <gazebo reference="front_cam_link">
+    <sensor name="front_camera" type="depth">
+      <always_on>1</always_on>
+      <visualize>1</visualize>
+      <update_rate>30</update_rate>
+      <camera>
+        <horizontal_fov>1.019272</horizontal_fov>
+        <image>
+          <width>640</width>
+          <height>480</height>
+          <format>B8G8R8</format>
+        </image>
+        <clip>
+          <near>0.2</near>
+          <far>8</far>
+        </clip>
+      </camera>
+      <plugin name="camera_front" filename="libgazebo_ros_camera.so">
+        <ros>
+          <namespace>${mp['namespace']}</namespace>
+        </ros>
+        <frame_name>${mp['namespace']}/front_cam_link</frame_name>
+        <camera_name>front</camera_name>
+        <hack_baseline>0.07</hack_baseline>
+        <min_depth>0.2</min_depth>
+        <max_depth>8.0</max_depth>
+      </plugin>
+    </sensor>
+  </gazebo>
+  <!-- <gazebo reference="front_cam_link">
     <sensor name="front_camera" type="camera">
       <always_on>1</always_on>
@@ -195,6 +224,4 @@
         <ros>
           <namespace>${mp['namespace']}</namespace>
-          <!-- <remapping>~/image_raw:=camera_front</remapping>
-          <remapping>~/camera_info:=camera_front_info</remapping> -->
         </ros>
         <frame_name>${mp['namespace']}/front_cam_link</frame_name>
@@ -203,7 +230,7 @@
       </plugin>
     </sensor>
-  </gazebo>
+  </gazebo> -->
   <!-- downward looking camera -->
-  <gazebo reference="bottom_cam_link">
+  <!-- <gazebo reference="bottom_cam_link">
     <sensor name="down_camera" type="camera">
       <always_on>1</always_on>
@@ -230,6 +257,4 @@
         <ros>
           <namespace>${mp['namespace']}</namespace>
-          <!-- <remapping>image_raw:=camera_bottom</remapping>
-          <remapping>camera_info:=camera_bottom_info</remapping> -->
         </ros>
         <frame_name>${mp['namespace']}/bottom_cam_link</frame_name>
@@ -238,5 +263,5 @@
       </plugin>
     </sensor>
-  </gazebo>
+  </gazebo> -->
   <gazebo reference="base_link">
     <sensor name="gps" type="gps">

Commit message: add std threshold slider

File: sjtu_drone_description/urdf/sjtu_drone.urdf (robot description, URDF)
Before this commit: robot sjtu_drone, 4 links, 3 joints
Links:
- link base_link: geometry collision mesh filename=file:///home/carlios/ros2_ws/install/sjtu_drone_description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; visual mesh filename=file:///home/carlios/ros2_ws/install/sjtu_drone_description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
Joints:
- joint front_cam_joint: origin xyz=0.2 0 0 rpy=0 0 0 -> xyz=0.2 0 0.45 rpy=0 0 0

Commit message: update camera orientation

File: sjtu_drone_description/urdf/sjtu_drone.urdf (robot description, URDF)
Before this commit: robot sjtu_drone, 4 links, 3 joints
Links:
- added link camera_link_optical
- link base_link: geometry collision mesh filename=file:///home/carlios/dev_ws/install/sjtu_drone_description/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; visual mesh filename=file:///home/carlios/dev_ws/install/sjtu_drone_description/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
Joints:
- added joint camera_optical_joint: type fixed, parent front_cam_link, child camera_link_optical, origin xyz=0 0 0 rpy=-1.5707963267948966 0 -1.5707963267948966

File: sjtu_drone_description/urdf/sjtu_drone.urdf.xacro (robot description, xacro)
@@ -7,4 +7,5 @@
   <xacro:arg name="y" default="0"/>
   <xacro:arg name="z" default="0.04"/>
+  <xacro name="pi" value="3.14159265359" />
   <!-- Need seperate property for xacro inorder processing -->
   <xacro:property name="params_path" value="$(arg params_path)"/>
@@ -51,4 +52,14 @@
   </joint>
   <link name="front_cam_link"/>
+  <joint name="camera_optical_joint" type="fixed">
+    <!-- these values have to be these values otherwise the gazebo camera
+          image won't be aligned properly with the frame it is supposedly
+          originating from -->
+    <origin xyz="0 0 0" rpy="${-pi/2} 0 ${-pi/2}" />
+    <parent link="front_cam_link" />
+    <child link="camera_link_optical" />
+  </joint>
+  <link name="camera_link_optical">
+  </link>
   <!-- <joint name="bottom_cam_joint" type="fixed">
     <origin rpy="0 ${M_PI/2} 0" xyz="0 0 0"/>
@@ -194,5 +205,5 @@
           <namespace>${mp['namespace']}</namespace>
         </ros>
-        <frame_name>${mp['namespace']}/front_cam_link</frame_name>
+        <frame_name>simple_drone/camera_link_optical</frame_name>
         <camera_name>front</camera_name>
         <hack_baseline>0.07</hack_baseline>
